File: ECAD/SatellitePump-2023/SatellitePump-2023.kicad_sch (KiCad schematic)
At the start: 18 parts, among them J1 Conn_02x05_Odd_Even, J10 Conn_01x03, J11 Conn_01x03, J2 Conn_01x02, J3 Conn_01x03, J4 Conn_01x03, J5 Conn_01x03, J6 Conn_01x03, J7 Conn_01x03, J8 Conn_01x03, J9 Conn_01x03

Commit message: New satellite Board
Parts:
- removed J7, J8: Conn_01x03, Footprints:PinHeader_3x01_P2.54mm_Horizontal, symbol Connector_Generic:Conn_01x03
- added D2, D3: LED_Small, LED_SMD:LED_1206_3216Metric_Pad1.42x1.75mm_HandSolder, symbol Device:LED_Small
- added D4, D5: D_Small, Diode_SMD:D_SMA_Handsoldering, symbol Device:D_Small
- added J7: CON_PUMP, Connector_Molex:Molex_KK-254_AE-6410-02A_1x02_P2.54mm_Vertical, symbol Connector_Generic:Conn_01x02
- added J8: CON_EV, Connector_Molex:Molex_KK-254_AE-6410-02A_1x02_P2.54mm_Vertical, symbol Connector_Generic:Conn_01x02
- added Q1, Q2: AO3400A, Package_TO_SOT_SMD:SOT-23, symbol Transistor_FET:AO3400A
- added R10, R8, R9: 220, Resistor_SMD:R_1206_3216Metric_Pad1.30x1.75mm_HandSolder, symbol Device:R_Small
- added R2, R3: 1k, Resistor_SMD:R_1206_3216Metric_Pad1.30x1.75mm_HandSolder, symbol Device:R_Small
- added R4, R5: 270R, Resistor_SMD:R_1206_3216Metric_Pad1.30x1.75mm_HandSolder, symbol Device:R_Small
- added R6, R7: 10K, Resistor_SMD:R_1206_3216Metric_Pad1.30x1.75mm_HandSolder, symbol Device:R_Small
Connections:
- net +5VP: now also D4.1 (K), D5.1 (K), J7.1 (Pin_1), J8.1 (Pin_1)
- net GND: now also J10.3 (Pin_3), J11.3 (Pin_3), J3.3 (Pin_3), J4.3 (Pin_3), J5.3 (Pin_3), J6.3 (Pin_3), J9.3 (Pin_3), D2.1 (K), D3.1 (K), Q1.2 (S), Q2.2 (S), R6.2, R7.2; no longer J10.1 (Pin_1), J11.1 (Pin_1), J3.1 (Pin_1), J4.1 (Pin_1), J5.1 (Pin_1), J6.1 (Pin_1), J9.1 (Pin_1)
- net IO_A_1: now also J1.8 (Pin_8), J11.1 (Pin_1); no longer J1.1 (Pin_1), J6.3 (Pin_3)
- net IO_A_2: now also J9.1 (Pin_1); no longer J9.3 (Pin_3)
- net IO_A_3: now also J1.1 (Pin_1), J6.1 (Pin_1); no longer J1.7 (Pin_7), J10.3 (Pin_3)
- net IO_A_4: now also J1.7 (Pin_7), J10.1 (Pin_1); no longer J1.8 (Pin_8), J11.3 (Pin_3)
- net IO_D_1: now also R8.2; no longer J3.3 (Pin_3)
- net IO_D_2: now also R9.2; no longer J4.3 (Pin_3)
- net IO_D_3: now also R10.2; no longer J5.3 (Pin_3)
- net IO_P_1: now also R2.1, R4.1
- net IO_P_2: now also R3.1, R5.1
- new net: D5.2 (A), J8.2 (Pin_2), Q2.3 (D)
- new net: J4.1 (Pin_1), R9.1
- new net: J5.1 (Pin_1), R10.1
- new net: Q1.1 (G), R4.2, R6.1
- new net: Q2.1 (G), R5.2, R7.1
- new net: J3.1 (Pin_1), R8.1
- new net: D4.2 (A), J7.2 (Pin_2), Q1.3 (D)
- new net: D2.2 (A), R2.2
- new net: D3.2 (A), R3.2
Other:
- note added: "Capteur de ventouse"
- note added: "Connecteur Servomoteurs"
- note added: "Gestion Pompe et EV"
- moved on the sheet: J10, J3, J4, J5, J6, J9
