File: ECAD/LidarBoard-2023/LidarBoard-2023.kicad_pcb (KiCad board)
At the start: 2 copper layers, 68.8 x 76.2 mm, 45 parts, among them J1 Serial_Strategy, J2 Serial_Lidar, J3 Conn_01x03, J4 Oled, U1 Teensy3.2, U2 AMS1117-3.3

Commit message: Live 141
Parts:
- moved J2 7.61 mm to (150.5, 111.6), turned to 180 degrees
- moved J1 7.61 mm to (163.2, 95.8), turned to -90 degrees
Connections:
- J1 pad 1: GND -> RX
- J1 pad 2: +5VP -> TX
- J1 pad 3: TX -> +5VP
- J1 pad 4: RX -> GND
- J2 pad 1: GND -> TX-Lidar
- J2 pad 2: +5VP -> LIDAR_PWM
- J2 pad 3: LIDAR_PWM -> +5VP
- J2 pad 4: TX-Lidar -> GND
Changed lines of the file:
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@@
   )
   (footprint "Connector_Molex:Molex_KK-254_AE-6410-04A_1x04_P2.54mm_Vertical" (layer "F.Cu")
-    (at 163.195 103.369103 90)
+    (at 163.195 95.758 -90)
     (descr "Molex KK-254 Interconnect System, old/engineering part number: AE-6410-04A example for new part number: 22-27-2041, 4 Pins (http://www.molex.com/pdm_docs/sd/022272021_sd.pdf), generated with kicad-footprint-generator")
     (tags "connector Molex KK-254 vertical")
@@
     (fp_line (start -0.562893 0) (end -1.27 0.5) (layer "F.Fab") (width 0.1))
     (fp_line (start 8.89 -2.92) (end -1.27 -2.92) (layer "F.Fab") (width 0.1))
-    (pad "1" thru_hole roundrect (at 0 0 90) (size 1.74 2.19) (drill 1.19) (layers *.Cu *.Mask) (roundrect_rratio 0.143678)
-      (net 18 "GND") (pinfunction "Pin_1") (pintype "passive"))
-    (pad "2" thru_hole oval (at 2.54 0 90) (size 1.74 2.19) (drill 1.19) (layers *.Cu *.Mask)
-      (net 1 "+5VP") (pinfunction "Pin_2") (pintype "passive"))
-    (pad "3" thru_hole oval (at 5.08 0 90) (size 1.74 2.19) (drill 1.19) (layers *.Cu *.Mask)
-      (net 25 "TX") (pinfunction "Pin_3") (pintype "passive"))
-    (pad "4" thru_hole oval (at 7.62 0 90) (size 1.74 2.19) (drill 1.19) (layers *.Cu *.Mask)
-      (net 26 "RX") (pinfunction "Pin_4") (pintype "passive"))
+    (pad "1" thru_hole roundrect (at 0 0 270) (size 1.74 2.19) (drill 1.19) (layers *.Cu *.Mask) (roundrect_rratio 0.143678)
+      (net 26 "RX") (pinfunction "Pin_1") (pintype "passive"))
+    (pad "2" thru_hole oval (at 2.54 0 270) (size 1.74 2.19) (drill 1.19) (layers *.Cu *.Mask)
+      (net 25 "TX") (pinfunction "Pin_2") (pintype "passive"))
+    (pad "3" thru_hole oval (at 5.08 0 270) (size 1.74 2.19) (drill 1.19) (layers *.Cu *.Mask)
+      (net 1 "+5VP") (pinfunction "Pin_3") (pintype "passive"))
+    (pad "4" thru_hole oval (at 7.62 0 270) (size 1.74 2.19) (drill 1.19) (layers *.Cu *.Mask)
+      (net 18 "GND") (pinfunction "Pin_4") (pintype "passive"))
     (model "${KIPRJMOD}/packages3D/Molex_KK-254_AE-6410-04A_1x04_P2.54mm_Vertical.wrl"
       (offset (xyz 0 0 0))
@@
   )
   (footprint "Connector_Molex:Molex_KK-254_AE-6410-04A_1x04_P2.54mm_Vertical" (layer "B.Cu")
-    (at 142.910974 111.553826)
+    (at 150.522577 111.550575 180)
     (descr "Molex KK-254 Interconnect System, old/engineering part number: AE-6410-04A example for new part number: 22-27-2041, 4 Pins (http://www.molex.com/pdm_docs/sd/022272021_sd.pdf), generated with kicad-footprint-generator")
     (tags "connector Molex KK-254 vertical")
@@
     (fp_line (start -1.27 2.92) (end -1.27 -2.88) (layer "B.Fab") (width 0.1))
     (fp_line (start -0.562893 0) (end -1.27 -0.5) (layer "B.Fab") (width 0.1))
-    (pad "1" thru_hole roundrect (at 0 0) (size 1.74 2.19) (drill 1.19) (layers *.Cu *.Mask) (roundrect_rratio 0.143678)
-      (net 18 "GND") (pinfunction "Pin_1") (pintype "passive"))
-    (pad "2" thru_hole oval (at 2.54 0) (size 1.74 2.19) (drill 1.19) (layers *.Cu *.Mask)
-      (net 1 "+5VP") (pinfunction "Pin_2") (pintype "passive"))
-    (pad "3" thru_hole oval (at 5.08 0) (size 1.74 2.19) (drill 1.19) (layers *.Cu *.Mask)
-      (net 27 "LIDAR_PWM") (pinfunction "Pin_3") (pintype "passive"))
-    (pad "4" thru_hole oval (at 7.62 0) (size 1.74 2.19) (drill 1.19) (layers *.Cu *.Mask)
-      (net 29 "TX-Lidar") (pinfunction "Pin_4") (pintype "passive"))
+    (pad "1" thru_hole roundrect (at 0 0 180) (size 1.74 2.19) (drill 1.19) (layers *.Cu *.Mask) (roundrect_rratio 0.143678)
+      (net 29 "TX-Lidar") (pinfunction "Pin_1") (pintype "passive"))
+    (pad "2" thru_hole oval (at 2.54 0 180) (size 1.74 2.19) (drill 1.19) (layers *.Cu *.Mask)
+      (net 27 "LIDAR_PWM") (pinfunction "Pin_2") (pintype "passive"))
+    (pad "3" thru_hole oval (at 5.08 0 180) (size 1.74 2.19) (drill 1.19) (layers *.Cu *.Mask)
+      (net 1 "+5VP") (pinfunction "Pin_3") (pintype "passive"))
+    (pad "4" thru_hole oval (at 7.62 0 180) (size 1.74 2.19) (drill 1.19) (layers *.Cu *.Mask)
+      (net 18 "GND") (pinfunction "Pin_4") (pintype "passive"))
     (model "${KIPRJMOD}/packages3D/Molex_KK-254_AE-6410-04A_1x04_P2.54mm_Vertical.wrl"
       (offset (xyz 0 0 0))
