File: ECAD/LidarBoard-2023/LidarBoard-2023.kicad_sch (KiCad schematic)
At the start: 17 parts, among them J1 Serial_Strategy, J2 Serial_Lidar, J3 Conn_01x03, J4 Oled, U1 Teensy3.2, U2 AMS1117-3.3

Commit message: Live 141
Connections:
- net +5VP: now also J1.3 (Pin_3), J2.3 (Pin_3); no longer J1.2 (Pin_2), J2.2 (Pin_2)
- net GND: now also J1.4 (Pin_4), J2.4 (Pin_4); no longer J1.1 (Pin_1), J2.1 (Pin_1)
- net LIDAR_PWM: now also J2.2 (Pin_2); no longer J2.3 (Pin_3)
- net RX: now also J1.1 (Pin_1); no longer J1.4 (Pin_4)
- net TX: now also J1.2 (Pin_2); no longer J1.3 (Pin_3)
- net TX-Lidar: now also J2.1 (Pin_1); no longer J2.4 (Pin_4)
Changed lines of the file:
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@@
     )
   )
-  (symbol (lib_id "Connector_Generic:Conn_01x04") (at 146.05 49.53 0) (unit 1)
+  (symbol (lib_id "Connector_Generic:Conn_01x04") (at 146.05 52.07 0) (mirror x) (unit 1)
     (in_bom yes) (on_board yes)
-    (property "Reference" "J2" (id 0) (at 148.59 49.5299 0)
+    (property "Reference" "J2" (id 0) (at 148.59 52.0701 0)
       (effects (font (size 1.27 1.27)) (justify left))
     )
-    (property "Value" "Serial_Lidar" (id 1) (at 139.7 43.18 0)
+    (property "Value" "Serial_Lidar" (id 1) (at 139.7 58.42 0)
       (effects (font (size 1.27 1.27)) (justify left))
     )
-    (property "Footprint" "Connector_Molex:Molex_KK-254_AE-6410-04A_1x04_P2.54mm_Vertical" (id 2) (at 146.05 49.53 0)
+    (property "Footprint" "Connector_Molex:Molex_KK-254_AE-6410-04A_1x04_P2.54mm_Vertical" (id 2) (at 146.05 52.07 0)
       (effects (font (size 1.27 1.27)) hide)
     )
-    (property "Datasheet" "~" (id 3) (at 146.05 49.53 0)
+    (property "Datasheet" "~" (id 3) (at 146.05 52.07 0)
       (effects (font (size 1.27 1.27)) hide)
     )
@@
     (pin "2")
   )
-  (symbol (lib_id "Connector_Generic:Conn_01x04") (at 146.05 30.48 0) (unit 1)
+  (symbol (lib_id "Connector_Generic:Conn_01x04") (at 146.05 33.02 0) (mirror x) (unit 1)
     (in_bom yes) (on_board yes)
-    (property "Reference" "J1" (id 0) (at 148.59 30.4799 0)
+    (property "Reference" "J1" (id 0) (at 148.59 33.0201 0)
       (effects (font (size 1.27 1.27)) (justify left))
     )
-    (property "Value" "Serial_Strategy" (id 1) (at 139.7 24.13 0)
+    (property "Value" "Serial_Strategy" (id 1) (at 139.7 39.37 0)
       (effects (font (size 1.27 1.27)) (justify left))
     )
-    (property "Footprint" "Connector_Molex:Molex_KK-254_AE-6410-04A_1x04_P2.54mm_Vertical" (id 2) (at 146.05 30.48 0)
+    (property "Footprint" "Connector_Molex:Molex_KK-254_AE-6410-04A_1x04_P2.54mm_Vertical" (id 2) (at 146.05 33.02 0)
       (effects (font (size 1.27 1.27)) hide)
     )
-    (property "Datasheet" "~" (id 3) (at 146.05 30.48 0)
+    (property "Datasheet" "~" (id 3) (at 146.05 33.02 0)
       (effects (font (size 1.27 1.27)) hide)
     )
