File: ECAD/TurbineBoard-2023/TurbineBoard-2023.kicad_pcb (KiCad board)
At the start: 2 copper layers, 58.3 x 108 mm, 26 parts, among them J1 Conn_02x05_Odd_Even, J10 Conn_01x03, J11 Conn_01x03, J2 Conn_01x02, J3 Conn_01x02, J4 Conn_01x03, J5 Conn_01x03, J6 Conn_01x02, J8 Conn_01x03, J9 Conn_01x03

Commit message: change dimensions and capacitor
Parts:
- C3: footprint Capacitor_THT:CP_Radial_D5.0mm_P2.00mm -> Capacitor_THT:CP_Radial_D16.0mm_P7.50mm
- moved J8 135.9 mm to (29.6, 118.5)
- moved J9 135.9 mm to (29.6, 128.2)
- moved J5 135.7 mm to (29.6, 108.2)
- moved J4 135.6 mm to (29.6, 98.2)
- moved J10 131.6 mm to (34.6, 139.2)
- moved J11 131.3 mm to (36.6, 153.2)
- moved D3 121.6 mm to (20.9, 75.0)
- moved J3 120.2 mm to (24.6, 80.7)
- moved LR1 101.0 mm to (29.0, 53.0)
- moved LR2 100.1 mm to (50.0, 53.0)
- moved D4 99.7 mm to (45.9, 75.0)
- moved J6 97.7 mm to (46.6, 80.7)
- moved R5 66.0 mm to (111.5, 125.0)
- moved R4 65.3 mm to (111.5, 121.0)
- moved R1 46.6 mm to (166.4, 90.0), turned to 180 degrees
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Other:
- board size 58.3 x 108 mm -> 55 x 110 mm

Commit message: update pcb - Aisler
Parts:
- added C1: 220uF 50V, Capacitor_THT:CP_Radial_D10.0mm_P5.00mm, F.Cu at (159.4, 131.4)
- C3: value 1200uF 50V -> 220uF 50V; footprint Capacitor_THT:CP_Radial_D16.0mm_P7.50mm -> Capacitor_THT:CP_Radial_D10.0mm_P5.00mm
- R1: value R_Small -> 1k
- R2: value R_Small -> 10k
- moved J5 148.3 mm to (157.5, 33.0), turned to 90 degrees
- moved J9 146.0 mm to (157.5, 57.7), turned to 90 degrees
- moved J3 143.9 mm to (168.3, 74.2), turned to 90 degrees
- moved D3 143.0 mm to (163.9, 75.0), turned to 90 degrees
- moved J10 139.1 mm to (147.3, 57.7), turned to 90 degrees
- moved J11 138.6 mm to (137.2, 57.7), turned to 90 degrees
- moved J8 137.4 mm to (137.2, 33.0), turned to 90 degrees
- moved J4 134.5 mm to (147.3, 33.0), turned to 90 degrees
- moved J6 122.1 mm to (168.2, 92.3), turned to 90 degrees
- moved D4 119.2 mm to (163.8, 92.9), turned to 90 degrees
- moved LR1 115.7 mm to (143.5, 69.8), turned to 90 degrees
- moved R5 101.1 mm to (161.0, 36.8), turned to 180 degrees
- moved LR2 99.7 mm to (143.5, 87.6), turned to 90 degrees
- moved R4 92.9 mm to (150.8, 36.8), turned to 180 degrees
- moved J1 53.2 mm to (129.5, 41.9), turned to 180 degrees
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Connections:
- D3 pad 1: Net-(D3-K) -> +5VP
- D4 pad 1: Net-(D4-K) -> +5VP
- J3 pad 1: Net-(D3-K) -> +5VP
- J6 pad 1: Net-(D4-K) -> +5VP
- LR1 pad 3: Net-(D3-K) -> +5VP
- LR2 pad 3: Net-(D4-K) -> +5VP
Routing:
- net +5VP: track 0.00 -> 206.5 mm
- net GND2: track 0.00 -> 77.4 mm
- net IO_D_1: track 0.00 -> 61.6 mm
- net +24V: track 0.00 -> 58.8 mm
- net IO_A_2: track 0.00 -> 52.0 mm
- net IO_P_2: track 0.00 -> 40.2 mm
- net IO_D_3: track 0.00 -> 34.1 mm
- net IO_A_3: track 0.00 -> 28.8 mm
- net IO_A_4: track 0.00 -> 25.4 mm
- net IO_D_2: track 0.00 -> 22.9 mm
- net IO_P_1: track 0.00 -> 21.9 mm
- net Net-(D3-A): track 0.00 -> 20.6 mm
- net Net-(D4-A): track 0.00 -> 20.3 mm
- net IO_A_1: track 0.00 -> 17.9 mm
- net Net-(J5-Pin_3): track 0.00 -> 3.81 mm
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- added copper zone on B.Cu, net GND
- added copper zone on F.Cu, net GND
Other:
- board size 55 x 110 mm -> 55 x 120 mm
