File: ECAD/TurbineBoard-2023/TurbineBoard-2023.kicad_pcb (KiCad board)
At the start: 2 copper layers, 55 x 120 mm, 27 parts, among them J1 Conn_02x05_Odd_Even, J10 Conn_01x03, J11 Conn_01x03, J2 Conn_01x02, J3 Conn_01x02, J4 Conn_01x03, J5 Conn_01x03, J6 Conn_01x02, J8 Conn_01x03, J9 Conn_01x03

Commit message: Fix turbine Board
Parts:
- removed D3, D4: D_Schottky_Small, Diode_THT:D_A-405_P10.16mm_Horizontal
- removed LR1, LR2: ~, LR7843:LR7843-Board
- added G***: LOGO, LOGO, F.Cu at (125.4, 47.0)
- added G***: LOGO, LOGO, F.Cu at (124.0, 87.0)
- added G***: LOGO, LOGO, F.Cu at (157.5, 59.6)
- added G***: LOGO, LOGO, F.Cu at (157.5, 34.8)
- added G***: LOGO, LOGO, F.Cu at (147.3, 34.8)
- added G***: LOGO, LOGO, F.Cu at (137.2, 34.8)
- added G***: LOGO, LOGO, F.Cu at (137.2, 59.5)
- added G***: LOGO, LOGO, F.Cu at (147.4, 59.6)
- added M1: ~, GA5A13-Board:GA5A13-Board, F.Cu at (146.0, 70.0)
- added M2: ~, GA5A13-Board:GA5A13-Board, F.Cu at (146.0, 88.0)
- added REF**: OSHW-Logo2_7.3x6mm_SilkScreen, Symbol:OSHW-Logo2_7.3x6mm_SilkScreen, F.Cu at (171.0, 35.5)
- moved J3 2.85 mm to (168.3, 71.4)
- moved J6 2.12 mm to (168.2, 94.4)
Connections:
- J2 pad 1: +24V -> GND2
- J2 pad 2: GND2 -> +24V
- J3 pad 1: +5VP -> Net-(J3-Pin_1)
- J6 pad 1: +5VP -> Net-(J6-Pin_1)
Routing:
- net GND: track 0.00 -> 33.5 mm
- net +5VP: track 206.5 -> 182.5 mm
- net Net-(J6-Pin_1): track 0.00 -> 22.3 mm
- net Net-(J3-Pin_1): track 0.00 -> 17.9 mm
- net Net-(J3-Pin_2): track 20.6 -> 16.4 mm
- net IO_P_1: track 21.9 -> 19.8 mm
- net IO_P_2: track 40.2 -> 38.9 mm
- net IO_A_2: track 52.0 -> 53.1 mm
Other:
- board text added: "+"
- board text added: "-"
- board text added: "Barbatronic"
- board text added: "Karibous 2022-23"
- board text added: "Motor"
- board text added: "SENSOR-01"
- board text added: "SENSOR-02"
- board text added: "SENSOR-03"
- board text added: "SENSOR-04"
- board text added: "SERVO-01"
- board text added: "SERVO-02"
- board text added: "Turbine"
