File: ECAD/TurbineBoard-2023/TurbineBoard-2023.kicad_sch (KiCad schematic)
At the start: 26 parts, among them J1 Conn_02x05_Odd_Even, J10 Conn_01x03, J11 Conn_01x03, J2 Conn_01x02, J3 Conn_01x02, J4 Conn_01x03, J5 Conn_01x03, J6 Conn_01x02, J8 Conn_01x03, J9 Conn_01x03

Commit message: change dimensions and capacitor
Parts:
- C3: footprint Capacitor_THT:CP_Radial_D5.0mm_P2.00mm -> Capacitor_THT:CP_Radial_D16.0mm_P7.50mm
Changed lines of the file:
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@@
       (effects (font (size 1.27 1.27)) (justify left))
     )
-    (property "Footprint" "Capacitor_THT:CP_Radial_D5.0mm_P2.00mm" (at 168.91 38.1 0)
+    (property "Footprint" "Capacitor_THT:CP_Radial_D16.0mm_P7.50mm" (at 168.91 38.1 0)
       (effects (font (size 1.27 1.27)) hide)
     )

Commit message: update pcb - Aisler
Parts:
- added C1: 220uF 50V, Capacitor_THT:CP_Radial_D10.0mm_P5.00mm, symbol Device:C_Polarized_Small
- C3: value 1200uF 50V -> 220uF 50V; footprint Capacitor_THT:CP_Radial_D16.0mm_P7.50mm -> Capacitor_THT:CP_Radial_D10.0mm_P5.00mm
- R1: value R_Small -> 1k
- R2: value R_Small -> 10k
Connections:
- net +24V: now also C1.1
- net +5VP: now also D3.1 (K), D4.1 (K), J3.1 (Pin_1), J6.1 (Pin_1), LR1.3 (+), LR2.3 (+)
- net GND2: now also C1.2
Other:
- moved on the sheet: C3, D1, D2, J2, R1, R2
