File: ECAD/TurbineBoard-2023/TurbineBoard-2023.kicad_sch (KiCad schematic)
At the start: 27 parts, among them J1 Conn_02x05_Odd_Even, J10 Conn_01x03, J11 Conn_01x03, J2 Conn_01x02, J3 Conn_01x02, J4 Conn_01x03, J5 Conn_01x03, J6 Conn_01x02, J8 Conn_01x03, J9 Conn_01x03

Commit message: Fix turbine Board
Parts:
- removed D3, D4: D_Schottky_Small, Diode_THT:D_A-405_P10.16mm_Horizontal, symbol Device:D_Schottky_Small
- removed LR1, LR2: ~, LR7843:LR7843-Board, symbol LR7843-Board:LR7843-Board
- added M1, M2: ~, GA5A13-Board:GA5A13-Board, symbol GA5A13-BOARD:GA5A13-Board
Connections:
- net +24V: now also J2.2 (Pin_2); no longer J2.1 (Pin_1)
- net +5VP: now also M1.3 (VIN+), M2.3 (VIN+); no longer J3.1 (Pin_1), J6.1 (Pin_1)
- net GND: now also M1.2 (GND), M1.4 (VIN-), M2.2 (GND), M2.4 (VIN-)
- net GND2: now also J2.1 (Pin_1); no longer J2.2 (Pin_2)
- net IO_P_1: now also M1.1 (PWM)
- net IO_P_2: now also M2.1 (PWM)
- net at J3.2 (Pin_2): now also M1.5 (VOUT+)
- net at J6.2 (Pin_2): now also M2.5 (VOUT+)
- new net: J3.1 (Pin_1), M1.6 (VOUT-)
- new net: J6.1 (Pin_1), M2.6 (VOUT-)
Other:
- moved on the sheet: J2, J3, J6
